File: mousekeyboard/mousekeyboard.kicad_pcb (KiCad board)
At the start: 2 copper layers, 97.5 x 67 mm, 12 parts, among them SW1 SW_Push, SW2 SW_Push, SW3 SW_Push, SW4 SW_Push, SW5 RotaryEncoder_Switch_MP, U1 MOUDLE-SEEEDUINO-XIAO, U2 ER_OLEDM0.91_1x-I2C

Commit message: overworking
Routing:
- net GND: track 209.9 -> 211.8 mm, vias 8 -> 11
Changed lines of the file:
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@@
+	)
+	(segment
+		(start 120.5 65)
+		(end 121.5 66)
+		(width 0.2)
+		(layer "F.Cu")
+		(net "GND")
+	)
+	(segment
+		(start 120 65)
+		(end 120.5 65)
+		(width 0.2)
+		(layer "F.Cu")
+		(net "GND")
 	)
 	(segment
@@
 	)
 	(via
+		(at 121.5 66)
+		(size 0.6)
+		(drill 0.3)
+		(layers "F.Cu" "B.Cu")
+		(net "GND")
+	)
+	(via
 		(at 124 77.5)
 		(size 0.6)
@@
 	(via
 		(at 124 92.5)
+		(size 0.6)
+		(drill 0.3)
+		(layers "F.Cu" "B.Cu")
+		(net "GND")
+	)
+	(via
+		(at 120 65)
 		(size 0.6)
 		(drill 0.3)
@@
 		(size 0.6)
 		(drill 0.3)
+		(layers "F.Cu" "B.Cu")
+		(net "GND")
+	)
+	(via
+		(at 121.5 66)
+		(size 0.6)
+		(drill 0.3)
