File: PCB/mousekeyboard/mousekeyboard.kicad_pcb (KiCad board)
At the start: 2 copper layers, 97.5 x 67 mm, 12 parts, among them SW1 SW_Push, SW2 SW_Push, SW3 SW_Push, SW4 SW_Push, SW5 RotaryEncoder_Switch_MP, U1 MOUDLE-SEEEDUINO-XIAO, U2 ER_OLEDM0.91_1x-I2C

Commit message: fixes
Parts:
- moved U1 8.88 mm to (110.5, 62.0)
Routing:
- net Net-(U1-PA6_A10_D10_MOSI): track 27.4 -> 51.9 mm, vias 0 -> 3
- net Net-(U1-PA8_A4_D4_SDA): track 55.3 -> 35.6 mm
- net Net-(U1-PA9_A5_D5_SCL): track 53.2 -> 33.8 mm
- net Net-(U1-PA5_A9_D9_MISO): track 31.2 -> 48.6 mm, vias 0 -> 4
- net +3.3V: track 11.5 -> 23.1 mm
- net Net-(U1-PA7_A8_D8_SCK): track 51.3 -> 61.0 mm, vias 2 -> 4
- net GND: track 211.8 -> 221.4 mm, vias 11 -> 6
- net Net-(U1-PB09_A7_D7_RX): track 72.2 -> 79.9 mm, vias 2 -> 3
- net Net-(U1-PA02_A0_D0): track 86.6 -> 80.2 mm, vias 2 -> 0
- net /re s2: track 117.4 -> 120.5 mm, vias 3 -> 4
- net Net-(U1-PA4_A1_D1): track 85.2 -> 87.9 mm, vias 2 -> 1
